File: eagle/Logging Controller.sch (EAGLE design)
At the start: 59 parts, among them J1 PWR IN, U1 ATMEGA328P_PDIP, U2 LCD-1602 3V3, U3 MCP1700-3302E/TO, X1 32.768kHz, 6pF, X2 16MHz

Commit message: tidied silk, adjusted some positions. Thick traces and ground fill
Parts:
- SJ1: value Bypass LDO for 3V3 supp -> Bypass LDOs
- renumbered U3 to LDO2
Changed lines of the file:
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@@
 <part name="D2" library="Astronomical Clocks" deviceset="DIODE-SCHOTTKY" device="DO-41" value="SR150"/>
 <part name="J1" library="Astronomical Clocks" deviceset="POWER_JACK" device="SLT" value="PWR IN"/>
-<part name="SJ1" library="Astronomical Clocks" deviceset="SOLDERJUMPER" device="NO" value="Bypass LDO for 3V3 supp"/>
+<part name="SJ1" library="Astronomical Clocks" deviceset="SOLDERJUMPER" device="NO" value="Bypass LDOs"/>
 <part name="U$2" library="Logging Controller" deviceset="MICROSD-HRS_DM3D" device=""/>
 <part name="U2" library="Logging Controller" deviceset="LCD-16X2" device="NOSILK" value="LCD-1602 3V3"/>
@@
 <part name="S2" library="Logging Controller" deviceset="SWITCH-MOMENTARY-2" device="OFF_BOARD_SPST" value="INPUT"/>
 <part name="S3" library="Logging Controller" deviceset="SWITCH-MOMENTARY-2" device="OFF_BOARD_SPST" value="BACKLIGHT"/>
-<part name="U3" library="Logging Controller" deviceset="MCP1700-3302E/TO" device=""/>
+<part name="LDO2" library="Logging Controller" deviceset="MCP1700-3302E/TO" device=""/>
 <part name="R9" library="Astronomical Clocks" deviceset="R-EU_" device="0204/7**" value="4k7"/>
 <part name="PAD1" library="Logging Controller" deviceset="WIREPAD" device="2,54/1,1" value="VIN"/>
@@
 <attribute name="VALUE" x="201.93" y="139.7" size="1.778" layer="96" rot="R90"/>
 </instance>
-<instance part="U3" gate="A" x="24.13" y="167.64" smashed="yes">
+<instance part="LDO2" gate="A" x="24.13" y="167.64" smashed="yes">
 <attribute name="NAME" x="19.431" y="171.4246" size="2.0828" layer="95" ratio="10" rot="SR0"/>
 <attribute name="VALUE" x="11.4046" y="158.9278" size="2.0828" layer="96" ratio="10" rot="SR0"/>
@@
 <wire x1="50.8" y1="156.21" x2="50.8" y2="149.86" width="0.1524" layer="91"/>
 <junction x="50.8" y="149.86"/>
-<pinref part="U3" gate="A" pin="VOUT"/>
+<pinref part="LDO2" gate="A" pin="VOUT"/>
 <wire x1="41.91" y1="165.1" x2="43.18" y2="165.1" width="0.1524" layer="91"/>
 <wire x1="43.18" y1="165.1" x2="43.18" y2="149.86" width="0.1524" layer="91"/>
@@
 <wire x1="-10.16" y1="124.46" x2="-10.16" y2="121.92" width="0.1524" layer="91"/>
 <wire x1="-10.16" y1="121.92" x2="-10.16" y2="114.3" width="0.1524" layer="91"/>
-<pinref part="U3" gate="A" pin="GND"/>
+<pinref part="LDO2" gate="A" pin="GND"/>
 <wire x1="6.35" y1="162.56" x2="-7.62" y2="162.56" width="0.1524" layer="91"/>
 <wire x1="-7.62" y1="162.56" x2="-7.62" y2="146.05" width="0.1524" layer="91"/>
@@
 <wire x1="8.89" y1="143.51" x2="15.24" y2="143.51" width="0.1524" layer="91"/>
 <wire x1="5.08" y1="134.62" x2="5.08" y2="165.1" width="0.1524" layer="91"/>
-<pinref part="U3" gate="A" pin="VIN"/>
+<pinref part="LDO2" gate="A" pin="VIN"/>
 <wire x1="5.08" y1="165.1" x2="6.35" y2="165.1" width="0.1524" layer="91"/>
 <pinref part="C11" gate="G$1" pin="+"/>

Commit message: v1.0.1 revision, esp fix power in pinout.
Parts:
- C4: value 10u -> 100u
- J1: device Astronomical Clocks:POWER_JACKSLT -> Astronomical Clocks:POWER_JACK**MJ-179PH
Other:
- note added: "CHOOSE ONE V-REG! MCP1700 with C4=10u gives lousy timekeeping on breadboard with a wall wart and caused hangs before WDT was used. XC6204 with C4=10u will not startup without a large cap on input (which can be removed after startup). Keeps good time on breadboard. XC6204 with C4=100u WILL startup fine and keeps good time."
- note added: "Logging Controller (RTC LCD SD) Version 1.0.1"
- note added: "Revisions: 1.0.1 - corrected footprint for PWR IN, uprated C4 to 100u, added SJ2 a/b on board, annotated SV1 pins on board"
- note removed: "CHOOSE ONE V-REG"
- note removed: "Logging Controller (RTC LCD SD) Version 1"
Changed lines of the file:
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@@
 <part name="JP2" library="Astronomical Clocks" deviceset="AVR-ISP-6" device="VERT" value="AVR-ISP"/>
 <part name="C3" library="Astronomical Clocks" deviceset="C-EU" device="025-024X044**100NF+22PF" value="100n"/>
-<part name="C4" library="Astronomical Clocks" deviceset="CPOL-EU" device="E2.5-5" value="10u"/>
+<part name="C4" library="Astronomical Clocks" deviceset="CPOL-EU" device="E2.5-5" value="100u"/>
 <part name="X2" library="Astronomical Clocks" deviceset="CRYSTAL*" device="-HC49U-V**16MHZ" value="16MHz"/>
 <part name="C5" library="Astronomical Clocks" deviceset="C-EU" device="025-024X044**100NF+22PF" value="22p"/>
@@
 <part name="LDO1" library="Astronomical Clocks" deviceset="XC6204/5" device="" value="XC6204B 3V3"/>
 <part name="D2" library="Astronomical Clocks" deviceset="DIODE-SCHOTTKY" device="DO-41" value="SR150"/>
-<part name="J1" library="Astronomical Clocks" deviceset="POWER_JACK" device="SLT" value="PWR IN"/>
+<part name="J1" library="Astronomical Clocks" deviceset="POWER_JACK" device="**MJ-179PH" value="PWR IN"/>
 <part name="SJ1" library="Astronomical Clocks" deviceset="SOLDERJUMPER" device="NO" value="Bypass LDOs"/>
 <part name="U$2" library="Logging Controller" deviceset="MICROSD-HRS_DM3D" device=""/>
@@
 <sheet>
 <plain>
-<text x="-22.86" y="78.74" size="3.81" layer="97">Adam Cooper, March 2014</text>
-<text x="-22.86" y="86.36" size="3.81" layer="97">Logging Controller (RTC LCD SD)
-Version 1</text>
+<text x="-25.4" y="73.66" size="3.81" layer="97">Adam Cooper, March 2014</text>
+<text x="-25.4" y="81.28" size="3.81" layer="97">Logging Controller (RTC LCD SD)
+Version 1.0.1</text>
 <text x="148.59" y="172.72" size="1.778" layer="97" rot="R90">Open=Run
 Closed=Set</text>
-<text x="19.05" y="195.58" size="1.778" layer="97">* - optional resistors
+<text x="52.07" y="213.36" size="1.778" layer="97">* - optional resistors
 omit if ATMega internal
 pull-ups enabled in code.
@@
 <text x="-25.4" y="134.62" size="1.778" layer="97">6V Max
 if MCP1700</text>
-<text x="-12.7" y="182.88" size="1.778" layer="97">** - optional for
+<text x="49.022" y="136.144" size="1.27" layer="97">** - optional for
 noise resistance</text>
 <text x="63.5" y="139.7" size="1.778" layer="97">**</text>
@@
 separately powered during
 programming.</text>
-<text x="10.16" y="172.72" size="1.778" layer="97" rot="R180">CHOOSE ONE
-V-REG</text>
+<text x="25.654" y="189.738" size="1.27" layer="97" rot="R180">CHOOSE ONE V-REG!
+MCP1700 with C4=10u gives lousy timekeeping
+on breadboard with a wall wart and caused
+hangs before WDT was used.
+XC6204 with C4=10u will not startup without a
+large cap on input (which can be removed after
+startup). Keeps good time on breadboard.
+XC6204 with C4=100u WILL startup fine and
+keeps good time.</text>
 <text x="208.28" y="157.48" size="1.778" layer="97" rot="R90">If LCD is not connected,
 run a 22k pull-down on E.
@@
 <text x="100.33" y="222.25" size="1.778" layer="97">CHOOSE: Serial Program
 or Bluetooth</text>
+<text x="-25.4" y="223.52" size="1.778" layer="97">Revisions:
+1.0.1 - corrected footprint for PWR IN,
+            uprated C4 to 100u,
+            added SJ2 a/b on board,
+            annotated SV1 pins on board</text>
 </plain>
 <instances>
@@
 <instance part="U1" gate="G$1" x="88.9" y="132.08"/>
 <instance part="GND2" gate="1" x="152.4" y="73.66"/>
-<instance part="GND3" gate="1" x="60.96" y="80.01"/>
+<instance part="GND3" gate="1" x="60.96" y="95.25"/>
 <instance part="GND4" gate="1" x="29.21" y="179.07"/>
 <instance part="GND5" gate="1" x="156.21" y="194.31"/>
@@
 <attribute name="VALUE" x="113.792" y="200.66" size="1.778" layer="96" rot="R90"/>
 </instance>
-<instance part="LOGO1" gate="G$1" x="-5.08" y="208.28"/>
+<instance part="LOGO1" gate="G$1" x="-10.16" y="106.68"/>
 <instance part="JP2" gate="G$1" x="123.19" y="78.74" smashed="yes">
 <attribute name="NAME" x="111.76" y="71.12" size="1.778" layer="95" ratio="10"/>
@@
 </instance>
 <instance part="X2" gate="X" x="59.69" y="127" rot="R90"/>
-<instance part="C5" gate="G$1" x="52.07" y="132.08" rot="R90"/>
+<instance part="C5" gate="G$1" x="52.07" y="132.08" smashed="yes" rot="R90">
+<attribute name="NAME" x="51.816" y="134.747" size="1.778" layer="95" rot="R180"/>
+<attribute name="VALUE" x="59.69" y="134.747" size="1.778" layer="96" rot="R180"/>
+</instance>
 <instance part="C6" gate="G$1" x="52.07" y="119.38" smashed="yes" rot="R90">
 <attribute name="NAME" x="51.689" y="114.554" size="1.778" layer="95" rot="R90"/>
@@
 <wire x1="66.04" y1="101.6" x2="66.04" y2="104.14" width="0.1524" layer="91"/>
 <pinref part="GND3" gate="1" pin="GND"/>
-<wire x1="60.96" y1="101.6" x2="60.96" y2="82.55" width="0.1524" layer="91"/>
+<wire x1="60.96" y1="101.6" x2="60.96" y2="97.79" width="0.1524" layer="91"/>
 <wire x1="0" y1="114.3" x2="0" y2="124.46" width="0.1524" layer="91"/>
 <pinref part="C4" gate="G$1" pin="-"/>
